File: hardware/kicad/mykovolt_devkit.kicad_sch (KiCad schematic)
At the start: 57 parts, among them J1 SWD_2x5, J2 Pressling, J3 Aux_I2C, J4 Sensor_In, Q1 SI1308EDL, U1 STM32L011F4Px, U2 BQ25570, U3 ST25DV04K, U4 MB85RC16, U5 PCF8523T, U6 FDC1004, X1 32.768kHz

Commit message: feat: fix all 57 PCB footprints, add copper zones, create firmware structure
PCB improvements:
- Fixed all 10 failing footprint names for KiCad 6 library compatibility
  (Package_SON, Inductor_SMD, Crystal, PinHeader, JST, THT cap, SOD)
- All 57 footprints now load successfully with pcbnew (0 warnings)
- Added GND copper pour on In1.Cu (inner layer 1)
- Added 3.3V copper pour on In2.Cu (inner layer 2)
- Pad net assignments from netlist (pads connected to correct nets)
- PCB size: 212662 bytes, 57 footprints, 2 copper zones

Firmware structure (STM32L011F4, bare-metal):
- firmware/README.md — architecture, pin map, power tree, I2C bus map
- Core/Inc/mykovolt.h — board definitions, pin mappings, I2C addresses
- Core/Inc/i2c_driver.h + .c — register-level I2C master (100kHz)
- Core/Inc/fdc1004.h — FDC1004 capacitance sensor driver header
- Core/Inc/st25dv04k.h — ST25DV04K NFC tag driver header
- Core/Src/main.c — app states: SLEEP → ACTIVE → NFC_ACCESS cycle
- CMakeLists.txt + cmake/arm-gcc-toolchain.cmake — build system
- Power-gated sleep with RTC wake, NFC mailbox data exchange

Generator: 57 components, 35 nets, 185 connections, 0 warnings, 0 errors
Verification: 22/22 checks pass
Parts:
- D2: footprint Package_TO_SOT_SMD:SOD-523 -> Diode_SMD:D_SOD-523
- J1: footprint Connector_Header:Header_2x05_P1.27mm_SMD -> Connector_PinHeader_1.27mm:PinHeader_2x05_P1.27mm_Vertical_SMD
- J2, J3: footprint Connector:JST_PH_B2B-PH-K_1x02_P2.0mm_Vertical -> Connector_JST:JST_PH_B2B-PH-K_1x02_P2.00mm_Vertical
- J4: footprint Connector_Header:Header_2x03_P1.27mm_SMD -> Connector_PinHeader_1.27mm:PinHeader_2x03_P1.27mm_Vertical_SMD
- L1: footprint Inductor_SMD:L_4x4mm_H2mm -> Inductor_SMD:L_Vishay_IFSC-1515AH_4x4x1.8mm
- L2: footprint Inductor_SMD:L_3x3mm_H1.5mm -> Inductor_SMD:L_Bourns-SRN4018
- SC1: footprint Capacitor_THT:CP_Radial_D8.0mm_P3.5mm -> Capacitor_THT:CP_Radial_D8.0mm_P3.50mm
- U6: footprint Package_SON:WSON-10-1EP_3x3mm_P0.5mm_EP1.6x2.0mm -> Package_SON:Texas_S-PWSON-N10
- X1: footprint Crystal:Crystal_SMD_3.2x1.5mm -> Crystal:Crystal_SMD_3215-2Pin_3.2x1.5mm
