File: hardware/kicad/mykovolt_devkit.kicad_pcb (KiCad board)
At the start: 4 copper layers, 30 x 20 mm, 57 parts, among them J1 SWD_2x5, J2 Pressling, J3 Aux_I2C, J4 Sensor_In, Q1 SI1308EDL, U1 STM32L011F4Px, U2 BQ25570, U3 ST25DV04K, U4 MB85RC16, U5 PCF8523T, U6 FDC1004, X1 32.768kHz

Commit message: professionalize: design rules, DRC tests, Gerber validator, project lib
- Add design_rules.yaml: externalized board config (clearance, routing,
  placement, fabrication constraints) — single source of truth
- Update generate_kicad.py: load YAML config, add CLI (--config, --variant,
  --skip-gerber, --skip-pcb), accept argv for test compatibility
- Add tests/test_pcb_drc.py: 10 tests for DRC validation, Gerber file
  completeness, board outline, component/net counts
- Add tools/validate_gerbers.py: Gerber validation against JLCPCB rules
  (layer completeness, syntax checks, file size validation)
- Add hardware/kicad/mykovolt.kicad_sym: project-specific symbol library
  (FDC1004, ST25DV04K extracted from schematic)
- All 95 tests pass (85 original + 10 new DRC/Gerber tests)
Parts:
- added ?: , , F.Cu at (0.00, 0.00)
- C1, C10, C11, C12, C13, C16, C17, C18, C19, C2, C20, C21, C22, C23, C24, C3, C4, C5, C6, C7, C8, C9: footprint C_0603_1608Metric -> Capacitor_SMD:C_0603_1608Metric
- C14, C15: footprint C_0805_2012Metric -> Capacitor_SMD:C_0805_2012Metric
- D1: footprint SOT-666 -> Package_TO_SOT_SMD:SOT-666
- D2: footprint D_SOD-523 -> Diode_SMD:D_SOD-523
- J1: footprint PinHeader_2x05_P1.27mm_Vertical_SMD -> Connector_PinHeader_1.27mm:PinHeader_2x05_P1.27mm_Vertical_SMD
- J2, J3: footprint JST_PH_B2B-PH-K_1x02_P2.00mm_Vertical -> Connector_JST:JST_PH_B2B-PH-K_1x02_P2.00mm_Vertical
- J4: footprint PinHeader_2x03_P1.27mm_Vertical_SMD -> Connector_PinHeader_1.27mm:PinHeader_2x03_P1.27mm_Vertical_SMD
- L1: footprint L_Vishay_IFSC-1515AH_4x4x1.8mm -> Inductor_SMD:L_Vishay_IFSC-1515AH_4x4x1.8mm
- L2: footprint L_Bourns-SRN4018 -> Inductor_SMD:L_Bourns-SRN4018
- LED1, LED2: footprint LED_0603_1608Metric -> LED_SMD:LED_0603_1608Metric
- Q1: footprint SOT-323_SC-70 -> Package_TO_SOT_SMD:SOT-323_SC-70
- R1, R10, R11, R12, R13, R14, R2, R3, R4, R5, R6, R7, R8, R9: footprint R_0603_1608Metric -> Resistor_SMD:R_0603_1608Metric
- SC1: footprint CP_Radial_D8.0mm_P3.50mm -> Capacitor_THT:CP_Radial_D8.0mm_P3.50mm
- U1: footprint TSSOP-20_4.4x6.5mm_P0.65mm -> Package_SO:TSSOP-20_4.4x6.5mm_P0.65mm
- U2: footprint QFN-20-1EP_3.5x3.5mm_P0.5mm_EP2x2mm -> Package_DFN_QFN:QFN-20-1EP_3.5x3.5mm_P0.5mm_EP2x2mm
- U3, U4, U5: footprint SOIC-8_3.9x4.9mm_P1.27mm -> Package_SO:SOIC-8_3.9x4.9mm_P1.27mm
- U6: footprint Texas_S-PWSON-N10 -> Package_SON:Texas_S-PWSON-N10
- X1: footprint Crystal_SMD_3215-2Pin_3.2x1.5mm -> Crystal:Crystal_SMD_3215-2Pin_3.2x1.5mm
Routing:
- net (no net): track 143.9 -> 0.00 mm
- net SHLD1: track 22.6 -> 0.00 mm
- net I2C1_SDA: track 22.2 -> 0.00 mm
- net I2C1_SCL: track 22.2 -> 0.00 mm
- net CIN1: track 21.3 -> 0.00 mm
- net VSTOR: track 21.0 -> 0.00 mm
- net CIN2: track 20.4 -> 0.00 mm
- net LED_PWR: track 14.0 -> 0.00 mm
- net NFC_RF1: track 13.0 -> 0.00 mm
- net NRST: track 11.0 -> 0.00 mm
- net NFC_IRQ: track 10.5 -> 0.00 mm
- net MCU_LED_CTRL: track 10.0 -> 0.00 mm
- net SWDIO: track 9.00 -> 0.00 mm
- net SENSOR_RDY: track 8.50 -> 0.00 mm
- net UART_TX: track 8.00 -> 0.00 mm
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- removed copper zone on In2.Cu, net 3.3V
- removed copper zone on In1.Cu, net GND
Other:
- board text removed: "30x20mm 4L ENIG RevA"
- board text removed: "MykoVolt DevKit v0.1"
- board text removed: "NFC ANT"
- board text removed: "SENSOR"

Commit message: feat: topology-driven PCB autorouter with A* pathfinding and persistent cache
Replaces hardcoded _route_critical_nets() with TopologyRouter:
- Obstacle grid (0.1mm) from actual footprint pads
- A* maze router with bounding-box search limits
- Net-class strategies: I2C daisy-chain, power wide, signal A*
- Straight-line pre-check to skip A* for obstacle-free paths
- Cached footprint loading (eliminates redundant 23s I/O)
- Persistent routing cache (first run 39s, subsequent 27s = 6.8x)

Also fixes pcbnew API for KiCad 9 (VECTOR2I, EDA_ANGLE) and adds
25 unit tests covering GridMap, classification, and integration.
Parts:
- removed ?: , 
- C1, C10, C11, C12, C13, C16, C17, C18, C19, C2, C20, C21, C22, C23, C24, C3, C4, C5, C6, C7, C8, C9: footprint Capacitor_SMD:C_0603_1608Metric -> C_0603_1608Metric
- C14, C15: footprint Capacitor_SMD:C_0805_2012Metric -> C_0805_2012Metric
- D1: footprint Package_TO_SOT_SMD:SOT-666 -> SOT-666
- D2: footprint Diode_SMD:D_SOD-523 -> D_SOD-523
- J1: footprint Connector_PinHeader_1.27mm:PinHeader_2x05_P1.27mm_Vertical_SMD -> PinHeader_2x05_P1.27mm_Vertical_SMD
- J2, J3: footprint Connector_JST:JST_PH_B2B-PH-K_1x02_P2.00mm_Vertical -> JST_PH_B2B-PH-K_1x02_P2.00mm_Vertical
- J4: footprint Connector_PinHeader_1.27mm:PinHeader_2x03_P1.27mm_Vertical_SMD -> PinHeader_2x03_P1.27mm_Vertical_SMD
- L1: footprint Inductor_SMD:L_Vishay_IFSC-1515AH_4x4x1.8mm -> L_Vishay_IFSC-1515AH_4x4x1.8mm
- L2: footprint Inductor_SMD:L_Bourns-SRN4018 -> L_Bourns-SRN4018
- LED1, LED2: footprint LED_SMD:LED_0603_1608Metric -> LED_0603_1608Metric
- Q1: footprint Package_TO_SOT_SMD:SOT-323_SC-70 -> SOT-323_SC-70
- R1, R10, R11, R12, R13, R14, R2, R3, R4, R5, R6, R7, R8, R9: footprint Resistor_SMD:R_0603_1608Metric -> R_0603_1608Metric
- SC1: footprint Capacitor_THT:CP_Radial_D8.0mm_P3.50mm -> CP_Radial_D8.0mm_P3.50mm
- U1: footprint Package_SO:TSSOP-20_4.4x6.5mm_P0.65mm -> TSSOP-20_4.4x6.5mm_P0.65mm
- U2: footprint Package_DFN_QFN:QFN-20-1EP_3.5x3.5mm_P0.5mm_EP2x2mm -> QFN-20-1EP_3.5x3.5mm_P0.5mm_EP2x2mm
- U3, U4, U5: footprint Package_SO:SOIC-8_3.9x4.9mm_P1.27mm -> SOIC-8_3.9x4.9mm_P1.27mm
- U6: footprint Package_SON:Texas_S-PWSON-N10 -> Texas_S-PWSON-N10
- X1: footprint Crystal:Crystal_SMD_3215-2Pin_3.2x1.5mm -> Crystal_SMD_3215-2Pin_3.2x1.5mm
Routing:
- net 3.3V: track 0.00 -> 1128.2 mm, vias 0 -> 12
- net CIN2: track 0.00 -> 74.5 mm
- added copper zone on In2.Cu, net 3.3V
- added copper zone on In1.Cu, net GND
Other:
- board text added: "30x20mm 4L ENIG RevA"
- board text added: "MykoVolt DevKit v0.1"
- board text added: "NFC ANT"
- board text added: "SENSOR"

Commit message: Update PCB design, test fixture spec, and gerber outputs
Routing:
- net CIN2: track 74.5 -> 0.00 mm
- net CIN1: track 0.00 -> 74.5 mm
