File: hardware/kicad/mykovolt_devkit.kicad_pcb (KiCad board)
At the start: 4 copper layers, 30 x 20 mm, 57 parts, among them J1 SWD_2x5, J2 Pressling, J3 Aux_I2C, J4 Sensor_In, Q1 SI1308EDL, U1 STM32L011F4Px, U2 BQ25570, U3 ST25DV04K, U4 MB85RC16, U5 PCF8523T, U6 FDC1004, X1 32.768kHz

Commit message: feat: export and CLI handle TestFixtureEntry (v2 FRAM entries)
Routing:
- net CIN1: track 74.5 -> 0.00 mm
- net CIN2: track 0.00 -> 74.5 mm

Commit message: refactor: move business-internal files, polish public repo
- Moved 17 business-sensitive files to private mykovolt-intern repo
- Fixed cross-references in docs/product/, simulation/README.md
- Updated README: docs entry, test count (175), added mykovolt/ CLI package
- Hardware/Gerbers: regeneration with VECTOR2I fix
Routing:
- net GND: track 0.00 -> 1128.2 mm, vias 0 -> 12
- net 3.3V: track 1128.2 -> 0.00 mm, vias 12 -> 0

Commit message: chore: add community files and polish public repo
- Added LICENSE (MIT), LICENSE_HARDWARE (CERN-OHL-P v2)
- Added CONTRIBUTING.md, CODE_OF_CONDUCT.md
- Added issue templates (bug report, feature request)
- Moved compliance_regulatory_roadmap.md → docs/technical/
- Removed empty docs/business/ directory
- Updated README license section with links
Routing:
- net GND: track 1128.2 -> 0.00 mm, vias 12 -> 0
- net 3.3V: track 0.00 -> 1128.2 mm, vias 0 -> 12
- net CIN2: track 74.5 -> 0.00 mm
- net CIN1: track 0.00 -> 74.5 mm
